File: Kicad Files/JuiceBox/JuiceBox.kicad_sch (KiCad schematic)
At the start: 13 parts, among them Q4 PMDT290UCE, Q5 PMDT290UCE, Q6 PMDT290UCE, Q7 PMDT290UCE, U1 LM22678TJ-5

Commit message: add convertor
Parts:
- added U2: LM5157RTER, LM5157RTER:QFN_57RTER_TEX, symbol LM5157RTER:LM5157RTER
Changed lines of the file:
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@@
+	)
+	(symbol
+		(lib_id "LM5157RTER:LM5157RTER")
+		(at 35.56 95.25 0)
+		(unit 1)
+		(exclude_from_sim no)
+		(in_bom yes)
+		(on_board yes)
+		(dnp no)
+		(fields_autoplaced yes)
+		(property "Reference" "U2"
+			(at 63.5 85.09 0)
+			(effects
+				(font
+					(size 1.524 1.524)
+				)
+			)
+		)
+		(property "Value" "LM5157RTER"
+			(at 63.5 87.63 0)
+			(effects
+				(font
+					(size 1.524 1.524)
+				)
+			)
+		)
+		(property "Footprint" "LM5157RTER:QFN_57RTER_TEX"
+			(at 35.56 95.25 0)
+			(effects
+				(font
+					(size 1.27 1.27)
+					(italic yes)
+				)
+				(hide yes)
+			)
+		)
+		(property "Datasheet" "https://www.ti.com/lit/gpn/lm5157"
+			(at 35.56 95.25 0)
+			(effects
+				(font
+					(size 1.27 1.27)
+					(italic yes)
+				)
+				(hide yes)
+			)
+		)
+		(property "Description" ""
+			(at 35.56 95.25 0)
+			(effects
+				(font
+					(size 1.27 1.27)
+				)
+				(hide yes)
+			)
+		)
+		(pin "3"
+		)
+		(pin "16"
+		)
+		(pin "4"
+		)
+		(pin "5"
+		)
+		(pin "12"
+		)
+		(pin "17"
+		)
+		(pin "10"
+		)
+		(pin "2"
+		)
+		(pin "9"
+		)
+		(pin "1"
+		)
+		(pin "14"
+		)
+		(pin "15"
+		)
+		(pin "11"
+		)
+		(pin "6"
+		)
+		(pin "7"
+		)
+		(pin "13"
+		)
+		(pin "8"
+		)
+		(instances
+			(project ""
+				(path "/83dc9953-a0fd-4bf5-b89c-ff1641ae0ce6"
+					(reference "U2")
+					(unit 1)
+				)
+			)
+		)
 	)
 	(symbol
